File: Uno4809/Freeduino4809.brd (EAGLE design)
At the start: 68.6 x 53.3 mm, 58 parts, among them J101 -, U1 ATMEGA4809, Y1 32768Hz

Commit message: Version 0.4 fix RX/TX, move UPDI pin
Parts:
- removed R2: 100k, my-rcl:R0805
- removed R4: 10k, my-rcl:R0805
- removed U1: ATMEGA4809, Arduino-ucs&SoCs:TQFP48
- added U2: ATMEGA4809-48SF, avr:LQFP48-SPARKFUN
- added W1, W2, W3, W4: WIRE-R6, mylib4:VIA6
- VERSION: value 0.3 -> 0.5
- moved UPDI 2.54 mm to (66.2, 22.9)
- moved RSTJ 1.51 mm to (23.3, 36.7)
- moved RSTJ1 1.46 mm to (25.1, 36.7)
- moved PA7 0.16 mm to (22.5, 44.2)
Connections:
- net DBG_RX: now also U2.8, USBMOD.RX, W1.P$1, W2.P$1; no longer U1.8, USBMOD.TX
- net DBG_TX: now also U2.9, USBMOD.TX, W3.P$1, W4.P$1; no longer U1.9, USBMOD.RX
- net GND: now also U2.15, U2.29, U2.43; no longer U1.15, U1.29, U1.43
- net LED_BUILTIN: now also U2.26; no longer U1.26
- net N$4: now also U2.34; no longer U1.34
- net N$5: now also U2.35; no longer U1.35
- net PA0: now also U2.44; no longer U1.44
- net PA1: now also U2.45; no longer U1.45
- net PA2: now also U2.46; no longer U1.46
- net PA3: now also U2.47; no longer U1.47
- net PA4: now also U2.48; no longer U1.48
- net PA5: now also U2.1; no longer U1.1
- net PA6: now also U2.2; no longer U1.2
- net PA7: now also U2.3; no longer U1.3
- net PB0: now also U2.4; no longer U1.4
- net PB1: now also U2.5; no longer U1.5
- net PB2: now also U2.6; no longer U1.6
- net PB3: now also U2.7; no longer U1.7
- net PC0: now also U2.10; no longer U1.10
- net PC1: now also U2.11; no longer U1.11
- net PC2: now also U2.12; no longer U1.12
- net PC3: now also U2.13; no longer U1.13
- net PC4: now also U2.16; no longer U1.16
- net PC5: now also U2.17; no longer U1.17
- net PC6: now also U2.18; no longer U1.18
- net PC7: now also U2.19; no longer U1.19
- net PD0: now also U2.20; no longer U1.20
- net PD1: now also U2.21; no longer U1.21
- net PD2: now also U2.22; no longer U1.22
- net PD3: now also U2.23; no longer U1.23
- net PD4: now also U2.24; no longer U1.24
- net PD5: now also U2.25; no longer U1.25
- net PD7: now also U2.27; no longer U1.27
- net PE0: now also U2.30; no longer U1.30
- net PE1: now also U2.31; no longer U1.31
- net PE2: now also U2.32; no longer U1.32
- net PE3: now also U2.33; no longer U1.33
- net PF2: now also U2.36; no longer U1.36
- net PF3: now also U2.37; no longer U1.37
- net PF4: now also U2.38; no longer U1.38
- net PF5: now also U2.39; no longer U1.39
- net TRG_RST: now also U2.40; no longer R2.1, U1.40
- net UPDI: now also U2.41; no longer R4.1, U1.41
- net VDD: now also U2.14, U2.28, U2.42; no longer R2.2, R4.2, U1.14, U1.28, U1.42
Routing:
- net TRG_RST: track 120.8 -> 115.2 mm
- net VDD: track 163.7 -> 161.9 mm, vias 4 -> 3
- net DBG_RX: track 43.5 -> 45.3 mm
- net UPDI: track 36.9 -> 36.0 mm
- net PA6: track 36.4 -> 37.2 mm
- net PA7: track 39.4 -> 39.9 mm
- net GND: track 14.7 -> 14.2 mm, vias 48 -> 49
Other:
- board text added: "20190805 by WestfW: Bump to V0.4. Fix reversed rxtx, add xover. Move UPDI pin."
- board text added: "20190812 by WestfW: Get rid of pull-up resistors on RST and UPDI."
- board text added: "20190814 by WestfW: change to Sparkfun LQFP package"
- board text removed: "100k"
- board text removed: "10k"
